File: detektor.kicad_sch (KiCad schematic)
At the start: 18 parts, among them J3 RCJ-011, Q1 BC548, Q2 BC558, Q3 BC548

Commit message: Return value of diode 1N4148
Parts:
- D1: value 1N4007 -> 1N4148
Changed lines of the file:
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@@
 			)
 		)
-		(property "Value" "1N4007"
+		(property "Value" "1N4148"
 			(at 175.26 96.774 0)
 			(show_name no)

Commit message: Change value of R1 to 4.2k
Parts:
- R6: value 3.9k -> 4.2k
Changed lines of the file:
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@@
 			)
 		)
-		(property "Value" "3.9k"
+		(property "Value" "4.2k"
 			(at 175.26 106.934 90)
 			(show_name no)
