File: detektor.kicad_sch (KiCad schematic)
At the start: 18 parts, among them J3 RCJ-011, Q1 BC548, Q2 BC558, Q3 BC548

Commit message: Change value of resistor R6 to 3.9k
Parts:
- R6: value 4.2k -> 3.9k
Changed lines of the file:
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@@
 			)
 		)
-		(property "Value" "4.2k"
+		(property "Value" "3.9k"
 			(at 175.26 106.934 90)
 			(show_name no)

Commit message: Change value of resistor R5 to 120K
Parts:
- R5: value 82k -> 120k
Changed lines of the file:
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@@
 			)
 		)
-		(property "Value" "82k"
+		(property "Value" "120k"
 			(at 165.1 83.82 90)
 			(show_name no)
