File: detektor.kicad_sch (KiCad schematic)
At the start: 18 parts, among them J3 RCJ-011, Q1 BC548, Q2 BC558, Q3 BC548

Commit message: Change diode to 1N4007
Parts:
- D1: value 1N4148 -> 1N4007
Changed lines of the file:
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@@
 			)
 		)
-		(property "Value" "1N4148"
+		(property "Value" "1N4007"
 			(at 175.26 96.774 0)
 			(show_name no)

Commit message: Change diode to 1N4148
Parts:
- D1: value 1N4007 -> 1N4148
Changed lines of the file:
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@@
 			)
 		)
-		(property "Value" "1N4007"
+		(property "Value" "1N4148"
 			(at 175.26 96.774 0)
 			(show_name no)

Commit message: Change value of resistor R7 to 1.3k
Parts:
- R7: value 1k -> 1.3k
Changed lines of the file:
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@@
 			)
 		)
-		(property "Value" "1k"
+		(property "Value" "1.3k"
 			(at 189.23 81.2799 0)
 			(show_name no)

Commit message: Change diode to 1N4007
Parts:
- D1: value 1N4148 -> 1N4007
Changed lines of the file:
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@@
 			)
 		)
-		(property "Value" "1N4148"
+		(property "Value" "1N4007"
 			(at 175.26 96.774 0)
 			(show_name no)
